File: pcb/holo clock 1.brd (EAGLE design)
At the start: 55.9 x 27.1 mm, 15 parts, among them IC2 7805DT, X1 POWERSUPPLY_DC21MMX

Commit message: final pcb
Parts:
- removed U$14, U$17, U$18: PLATED-SCREW, Sanguinololu:PLATEDSCREW
- added C24, C26: 22pf, SparkFun:0805
- added Q5: (no value), crystal:HC49/S
- moved R1 27.0 mm to (43.0, 23.0)
- moved IC2 3.16 mm to (7.16, 20.1)
- moved U$5 3.16 mm to (28.0, 19.0)
- moved C8 3.00 mm to (2.70, 15.2)
- moved S2 2.55 mm to (47.9, 21.7)
- moved C4 2.24 mm to (12.8, 13.9)
- moved R2 2.24 mm to (36.0, 20.0), turned to 180 degrees
- moved LED3 2.00 mm to (39.0, 24.0)
- moved ULN2803 2.00 mm to (41.3, 8.70)
- moved JP2 1.00 mm to (25.0, 5.00)
- moved X1 1.00 mm to (4.54, 5.59)
Connections:
- new net N$80: C26.2, Q5.2, U$5.4
- new net N$81: C24.2, Q5.1, U$5.5
- net GND: now also C24.1, C26.1; no longer U$14.GND, U$17.GND, U$18.GND
Routing:
- net !RESET: track 23.4 -> 45.3 mm, vias 1 -> 0
- net 5V: track 63.5 -> 84.4 mm, vias 1 -> 0
- net N$80: track 0.00 -> 20.2 mm
- net N$81: track 0.00 -> 19.0 mm
- net PWRIN: track 64.6 -> 81.8 mm
- net SCLK: track 10.2 -> 22.8 mm, vias 1 -> 0
- net N$8: track 38.0 -> 30.4 mm
- net N$2: track 35.0 -> 28.4 mm
- net D1: track 39.1 -> 33.8 mm
- net GND: track 0.00 -> 3.10 mm, vias 1 -> 5
- net D2: track 31.8 -> 28.9 mm
- net MOSI: track 10.1 -> 11.9 mm
- net N$7: track 2.78 -> 4.08 mm
- net N$5: track 10.2 -> 8.94 mm
- net N$1: track 13.0 -> 12.0 mm
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